File: onizuka.kicad_pcb (KiCad board)
At the start: 2 copper layers, 50 x 50 mm, 26 parts, among them IC1 FT232RQ, IC2 ADCMP371, P1 USB_OTG, P2 CONN_01X10, Q1 Q_PMOS_DGS, SW1 SWITCH_INV, U1 LD1117S33TR

Commit message: more shenanigans
Parts:
- added P3: EXTRA, Pin_Headers:Pin_Header_Angled_1x04, F.Cu at (65.7, 36.7)
- P2: value CONN_01X10 -> FTDI; footprint Pin_Headers:Pin_Header_Angled_1x10 -> Pin_Headers:Pin_Header_Angled_1x06
- moved P1 55.9 mm to (40.9, 19.3), turned to 180 degrees
- moved IC1 4.10 mm to (42.2, 28.3), turned to 0 degrees
Connections:
- IC1 pad 10: Net-(IC1-Pad10) -> (no net)
- IC1 pad 12: Net-(IC1-Pad12) -> (no net)
- IC1 pad 13: Net-(IC1-Pad13) -> (no net)
- IC1 pad 18: Net-(IC1-Pad18) -> (no net)
- IC1 pad 2: Net-(IC1-Pad2) -> /RXD
- IC1 pad 23: Net-(IC1-Pad23) -> (no net)
- IC1 pad 25: Net-(IC1-Pad25) -> (no net)
- IC1 pad 27: Net-(IC1-Pad27) -> (no net)
- IC1 pad 28: Net-(IC1-Pad28) -> (no net)
- IC1 pad 29: Net-(IC1-Pad29) -> (no net)
- IC1 pad 3: Net-(IC1-Pad3) -> /RI
- IC1 pad 30: Net-(IC1-Pad30) -> /TXD
- IC1 pad 31: Net-(IC1-Pad31) -> /DTR
- IC1 pad 32: Net-(IC1-Pad32) -> /RTS
- IC1 pad 5: Net-(IC1-Pad5) -> (no net)
- IC1 pad 6: Net-(IC1-Pad6) -> /DSR
- IC1 pad 7: Net-(IC1-Pad7) -> /DCD
- IC1 pad 8: Net-(IC1-Pad8) -> /CTS
- IC1 pad 9: Net-(IC1-Pad9) -> (no net)
- P1 pad 4: Net-(P1-Pad4) -> (no net)
- P2 pad 1: /PWROUT -> GND
- P2 pad 2: Net-(IC1-Pad30) -> /CTS
- P2 pad 3: Net-(IC1-Pad2) -> /PWROUT
- P2 pad 4: Net-(IC1-Pad32) -> /TXD
- P2 pad 5: Net-(IC1-Pad8) -> /RXD
- P2 pad 6: Net-(IC1-Pad31) -> /RTS
Routing:
- net Net-(IC1-Pad30): track 12.0 -> 0.00 mm, vias 2 -> 0
- net Net-(IC1-Pad31): track 9.22 -> 0.00 mm
- net Net-(IC1-Pad32): track 5.56 -> 0.00 mm
- net Net-(IC1-Pad2): track 4.89 -> 0.00 mm
- net /PWROUT: track 6.80 -> 3.07 mm
- net Net-(IC1-Pad6): track 2.66 -> 0.00 mm
- net Net-(IC1-Pad7): track 2.60 -> 0.00 mm
- net Net-(IC1-Pad8): track 2.46 -> 0.00 mm
- net /RTS: track 0.00 -> 1.32 mm
- removed copper zone on B.Cu, net GND
