File: master-board/onizuka.kicad_pcb (KiCad board)
At the start: 2 copper layers, 25.5 x 16 mm, 30 parts, among them IC1 FT232RQ, IC2 ADCMP371, P1 USB_OTG, P2 FTDI, Q1 Q_PMOS_GSD, SW1 SWITCH_INV, U1 MIC5353-3.3YMT

Commit message: Add board names revisions and emails.
Other:
- board text added: "Onizuka V0.1 01/06/16 board@harkonen.net"
Changed lines of the file:
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@@
     (area 42.924999 19.924999 68.575001 36.075001)
     (thickness 1.6)
-    (drawings 6)
+    (drawings 7)
     (tracks 282)
     (zones 0)
@@
     )
   )
+  (gr_text "Onizuka\nV0.1 01/06/16\nboard@harkonen.net" (at 52.197 31.369) (layer B.SilkS)
+    (effects (font (size 1 1) (thickness 0.15)) (justify mirror))
+  )
   (gr_text 3v3 (at 49 25) (layer F.SilkS)

Commit message: Updated switch
Parts:
- SW1: value SWITCH_INV -> SPDT; footprint Buttons_Switches_ThroughHole:SW_Micro_SPST -> Wurth:450301014042
- moved R9 2.34 mm to (44.4, 23.0), turned to 0 degrees
- moved R4 2.29 mm to (44.7, 21.3)
- moved C4 2.29 mm to (52.5, 29.6), turned to 270 degrees
- moved C3 1.08 mm to (53.7, 28.4), turned to 90 degrees
- moved SW1 1.01 mm to (48.0, 26.7)
- moved C2 0.39 mm to (50.5, 23.9)
- moved C5 0.38 mm to (49.3, 21.5)
- moved C6 0.38 mm to (50.5, 21.5)
Connections:
- SW1 pad 1: +5V -> /VCCIO
- SW1 pad 2: /VCCIO -> +5V
Routing:
- net +5V: track 42.5 -> 47.8 mm
- net GND: track 39.1 -> 36.9 mm, vias 12 -> 13
- net /PWREN: track 20.3 -> 22.3 mm
- net Net-(C5-Pad2): track 6.07 -> 4.73 mm
- net +3V3: track 5.61 -> 6.66 mm

Commit message: Poked around, fixed minor bug, tweaked silk slightly.
Parts:
- moved R9 0.09 mm to (44.5, 22.9), turned to 180 degrees
Connections:
- IC1 pad 10: (no net) -> Net-(IC1-Pad10)
- IC1 pad 12: (no net) -> Net-(IC1-Pad12)
- IC1 pad 13: (no net) -> Net-(IC1-Pad13)
- IC1 pad 18: (no net) -> Net-(IC1-Pad18)
- IC1 pad 23: (no net) -> Net-(IC1-Pad23)
- IC1 pad 25: (no net) -> Net-(IC1-Pad25)
- IC1 pad 27: (no net) -> Net-(IC1-Pad27)
- IC1 pad 28: (no net) -> Net-(IC1-Pad28)
- IC1 pad 29: (no net) -> Net-(IC1-Pad29)
- IC1 pad 5: (no net) -> Net-(IC1-Pad5)
- IC1 pad 9: (no net) -> Net-(IC1-Pad9)
- P1 pad 4: (no net) -> Net-(P1-Pad4)
- P2 pad 10: (no net) -> Net-(P2-Pad10)
- P2 pad 12: (no net) -> Net-(P2-Pad12)
- R9 pad 1: +5V -> /VCCIO
- U1 pad 5: (no net) -> Net-(U1-Pad5)
Routing:
- net +5V: track 47.8 -> 43.5 mm
- net /PWREN: track 22.3 -> 23.6 mm
- net /VCCIO: track 28.1 -> 29.3 mm

Commit message: Many faffing, new ESP stuff.
Parts:
- P2: footprint Pin_Headers:Pin_Header_Angled_2x06 -> Socket_Strips:Socket_Strip_Angled_2x06
- moved P2 12.6 mm to (62.0, 34.3), turned to 90 degrees
Connections:
- P2 pad 1: GND -> /RTS
- P2 pad 10: Net-(P2-Pad10) -> /DSR
- P2 pad 11: /RTS -> GND
- P2 pad 12: Net-(P2-Pad12) -> /DTR
- P2 pad 2: /DTR -> Net-(P2-Pad2)
- P2 pad 3: /CTS -> /RXD
- P2 pad 4: /DSR -> Net-(P2-Pad4)
- P2 pad 5: /PWROUT -> /TXD
- P2 pad 6: /DCD -> /RI
- P2 pad 7: /TXD -> /PWROUT
- P2 pad 8: /RI -> /DCD
- P2 pad 9: /RXD -> /CTS
Other:
- board size 25.5 x 16 mm -> 23.5 x 16 mm

Commit message: Various shuffling, adding farnell part numbers.
Parts:
- moved R1 0.38 mm to (55.8, 33.5)
- moved C3 0.06 mm to (53.7, 28.4)
Connections:
- IC1 pad 10: Net-(IC1-Pad10) -> (no net)
- IC1 pad 12: Net-(IC1-Pad12) -> (no net)
- IC1 pad 13: Net-(IC1-Pad13) -> (no net)
- IC1 pad 18: Net-(IC1-Pad18) -> (no net)
- IC1 pad 23: Net-(IC1-Pad23) -> (no net)
- IC1 pad 25: Net-(IC1-Pad25) -> (no net)
- IC1 pad 27: Net-(IC1-Pad27) -> (no net)
- IC1 pad 28: Net-(IC1-Pad28) -> (no net)
- IC1 pad 29: Net-(IC1-Pad29) -> (no net)
- IC1 pad 5: Net-(IC1-Pad5) -> (no net)
- IC1 pad 9: Net-(IC1-Pad9) -> (no net)
- P1 pad 4: Net-(P1-Pad4) -> (no net)
- P2 pad 12: /DTR -> (no net)
- P2 pad 2: Net-(P2-Pad2) -> (no net)
- P2 pad 4: Net-(P2-Pad4) -> /DTR
- U1 pad 5: Net-(U1-Pad5) -> (no net)
Routing:
- net /DTR: track 24.1 -> 11.8 mm
- net Net-(D1-Pad1): track 1.18 -> 1.80 mm
Other:
- board size 23.5 x 16 mm -> 22.8 x 16 mm
