File: master-board/onizuka.kicad_pcb (KiCad board)
At the start: 2 copper layers, 22.8 x 16 mm, 30 parts, among them IC1 FT232RQ, IC2 ADCMP371, P1 USB_OTG, P2 FTDI, Q1 Q_PMOS_GSD, SW1 SPDT, U1 MIC5353-3.3YMT

Commit message: Final tweaks, more farnell part numbers, BOM, gerbers
Parts:
- R4: value 1K -> 1k
Other:
- board text added: "Onizuka V1.0 04/06/16 board@harkonen.net"
- board text removed: "Onizuka V0.1 01/06/16 board@harkonen.net"
Changed lines of the file:
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@@
-(kicad_pcb (version 4) (host pcbnew 4.1.0-alpha+201605292346+6852~44~ubuntu16.04.1-product)
+(kicad_pcb (version 4) (host pcbnew "(2016-06-01 BZR 6870, Git 0ccd3bb)-product")
   (general
     (links 75)
     (no_connects 0)
-    (area 42.924999 19.924999 65.825001 36.075001)
+    (area 39.357738 16.785 75.351001 37.9375)
     (thickness 1.6)
     (drawings 11)
-    (tracks 303)
+    (tracks 306)
     (zones 0)
     (modules 30)
@@
     (visible_elements 7FFFFF7F)
     (pcbplotparams
-      (layerselection 0x00030_80000001)
-      (usegerberextensions false)
+      (layerselection 0x010fc_ffffffff)
+      (usegerberextensions true)
       (excludeedgelayer true)
-      (linewidth 0.100000)
+      (linewidth 0.150000)
       (plotframeref false)
       (viasonmask false)
@@
       (outputformat 1)
       (mirror false)
-      (drillshape 1)
+      (drillshape 0)
       (scaleselection 1)
-      (outputdirectory ""))
+      (outputdirectory gerbers/))
   )
   (net 0 "")
@@
       (effects (font (size 1 1) (thickness 0.15)))
     )
-    (fp_text value 1K (at 0 1.8 270) (layer F.Fab) hide
+    (fp_text value 1k (at 0 1.8 270) (layer F.Fab) hide
       (effects (font (size 1 1) (thickness 0.15)))
     )
@@
   (gr_arc (start 65.25 35.5) (end 65.75 35.5) (angle 90) (layer Edge.Cuts) (width 0.15))
   (gr_arc (start 65.25 20.5) (end 65.25 20) (angle 90) (layer Edge.Cuts) (width 0.15))
-  (gr_text "Onizuka\nV0.1 01/06/16\nboard@harkonen.net" (at 52.197 31.369) (layer B.SilkS)
+  (gr_text "Onizuka\nV1.0 04/06/16\nboard@harkonen.net" (at 52.197 31.369) (layer B.SilkS)
     (effects (font (size 1 1) (thickness 0.15)) (justify mirror))
   )
@@
   (segment (start 59.5065 31.115) (end 61.2775 31.115) (width 0.25) (layer F.Cu) (net 16))
   (segment (start 61.2775 31.115) (end 61.976 31.8135) (width 0.25) (layer F.Cu) (net 16))
+  (segment (start 59.3865 30.595) (end 59.9365 30.595) (width 0.25) (layer F.Cu) (net 17))
+  (segment (start 59.9365 30.595) (end 60.132899 30.398601) (width 0.25) (layer F.Cu) (net 17))
+  (segment (start 60.132899 30.398601) (end 63.327399 30.398601) (width 0.25) (layer F.Cu) (net 17))
+  (segment (start 63.327399 30.398601) (end 63.652401 30.073599) (width 0.25) (layer F.Cu) (net 17))
+  (segment (start 63.652401 30.073599) (end 64.516 29.21) (width 0.25) (layer F.Cu) (net 17))
   (segment (start 59.4865 30.595) (end 59.4985 30.607) (width 0.25) (layer F.Cu) (net 17))
-  (segment (start 59.4985 30.607) (end 63.1825 30.607) (width 0.25) (layer F.Cu) (net 17))
-  (segment (start 63.1825 30.607) (end 64.516 29.2735) (width 0.25) (layer F.Cu) (net 17))
-  (segment (start 59.4865 29.095) (end 60.44 29.095) (width 0.25) (layer F.Cu) (net 18))
-  (segment (start 60.44 29.095) (end 61.5315 28.0035) (width 0.25) (layer F.Cu) (net 18))
+  (segment (start 59.3865 29.095) (end 60.33187 29.095) (width 0.25) (layer F.Cu) (net 18))
+  (segment (start 60.33187 29.095) (end 61.568269 27.858601) (width 0.25) (layer F.Cu) (net 18))
+  (segment (start 61.568269 27.858601) (end 62.565399 27.858601) (width 0.25) (layer F.Cu) (net 18))
+  (segment (start 62.565399 27.858601) (end 63.246 27.178) (width 0.25) (layer F.Cu) (net 18))
   (segment (start 63.246 25.4635) (end 64.516 24.1935) (width 0.25) (layer F.Cu) (net 18))
   (segment (start 63.246 27.178) (end 63.246 25.4635) (width 0.25) (layer F.Cu) (net 18))
-  (segment (start 62.4205 28.0035) (end 63.246 27.178) (width 0.25) (layer F.Cu) (net 18))
-  (segment (start 61.5315 28.0035) (end 62.4205 28.0035) (width 0.25) (layer F.Cu) (net 18))
-  (segment (start 59.4865 28.595) (end 60.051 28.595) (width 0.25) (layer F.Cu) (net 19))
+  (segment (start 60.5155 28.0035) (end 63.246 28.0035) (width 0.25) (layer B.Cu) (net 19))
+  (segment (start 59.3865 28.595) (end 59.924 28.595) (width 0.25) (layer F.Cu) (net 19))
+  (segment (start 59.924 28.595) (end 60.5155 28.0035) (width 0.25) (layer F.Cu) (net 19))
+  (via (at 60.5155 28.0035) (size 0.6) (drill 0.4) (layers F.Cu B.Cu) (net 19))
   (segment (start 63.246 28.0035) (end 64.516 26.7335) (width 0.25) (layer B.Cu) (net 19))
-  (segment (start 61.2775 28.0035) (end 63.246 28.0035) (width 0.25) (layer B.Cu) (net 19))
-  (segment (start 60.96 27.686) (end 61.2775 28.0035) (width 0.25) (layer B.Cu) (net 19))
-  (via (at 60.96 27.686) (size 0.6) (drill 0.4) (layers F.Cu B.Cu) (net 19))
-  (segment (start 60.051 28.595) (end 60.96 27.686) (width 0.25) (layer F.Cu) (net 19))
-  (segment (start 59.4865 28.095) (end 59.5985 28.095) (width 0.25) (layer F.Cu) (net 20))
-  (segment (start 59.5985 28.095) (end 60.7695 26.924) (width 0.25) (layer F.Cu) (net 20))
-  (segment (start 60.7695 26.924) (end 60.7695 25.4) (width 0.25) (layer F.Cu) (net 20))
-  (segment (start 60.7695 25.4) (end 61.976 24.1935) (width 0.25) (layer F.Cu) (net 20))
+  (segment (start 59.3865 28.095) (end 59.498998 28.095) (width 0.25) (layer F.Cu) (net 20))
+  (segment (start 59.498998 28.095) (end 60.787399 26.806599) (width 0.25) (layer F.Cu) (net 20))
+  (segment (start 60.787399 26.806599) (end 60.787399 25.418103) (width 0.25) (layer F.Cu) (net 20))
+  (segment (start 60.787399 25.418103) (end 61.976 24.229502) (width 0.25) (layer F.Cu) (net 20))
+  (segment (start 61.976 24.229502) (end 61.976 24.13) (width 0.25) (layer F.Cu) (net 20))
   (segment (start 60.6425 35.56) (end 60.3885 35.56) (width 0.25) (layer B.Cu) (net 21))
   (segment (start 57.8365 33.008) (end 59.944 35.1155) (width 0.25) (layer F.Cu) (net 21))

Commit message: Updated Thin MLF footprint, regenned gerbers
Other:
- rule pad_to_mask_clearance: 0 -> 0.06
Changed lines of the file:
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@@
     (links 75)
     (no_connects 0)
-    (area 39.357738 16.785 75.351001 37.9375)
+    (area 42.924999 19.924999 65.825001 36.075001)
     (thickness 1.6)
     (drawings 11)
@@
     (pad_size 3.6576 2.032)
     (pad_drill 0)
-    (pad_to_mask_clearance 0)
+    (pad_to_mask_clearance 0.06)
     (aux_axis_origin 0 0)
     (visible_elements 7FFFFF7F)
@@
     )
   )
-  (module Housings_MLF:Thin_MLF_6_1.6mm_0.5mm_pitch (layer F.Cu)
-    (at 46.0375 30.48)
-    (fp_text reference U1 (at 0 1.7) (layer F.SilkS) hide
-      (effects (font (size 1 1) (thickness 0.15)))
-    )
-    (fp_text value MIC5353-3.3YMT (at 0 -1.9) (layer F.Fab) hide
-      (effects (font (size 1 1) (thickness 0.15)))
-    )
-    (fp_line (start 1 -1) (end 1 1) (layer F.CrtYd) (width 0.05))
-    (fp_line (start 1 1) (end -1 1) (layer F.CrtYd) (width 0.05))
-    (fp_line (start -1 1) (end -1 -1) (layer F.CrtYd) (width 0.05))
-    (fp_line (start -1 -1) (end 1 -1) (layer F.CrtYd) (width 0.05))
-    (fp_line (start -0.8 -0.8) (end 0 -0.8) (layer F.SilkS) (width 0.15))
-    (fp_line (start 0.4 0.8) (end 0 0.8) (layer F.SilkS) (width 0.15))
-    (pad 4 smd rect (at 0.7 0.5) (size 0.35 0.25) (layers F.Cu F.Paste F.Mask)
-      (net 15 +3V3) (solder_mask_margin 0.06))
-    (pad 5 smd rect (at 0.7 0) (size 0.35 0.25) (layers F.Cu F.Paste F.Mask)
-      (solder_mask_margin 0.06))
-    (pad 6 smd rect (at 0.7 -0.5) (size 0.35 0.25) (layers F.Cu F.Paste F.Mask)
-      (net 27 "Net-(C9-Pad2)") (solder_mask_margin 0.06))
-    (pad 3 smd rect (at -0.7 0.5) (size 0.35 0.25) (layers F.Cu F.Paste F.Mask)
-      (net 3 +5V) (solder_mask_margin 0.06))
-    (pad 1 smd rect (at -0.7 -0.5) (size 0.35 0.25) (layers F.Cu F.Paste F.Mask)
-      (net 3 +5V) (solder_mask_margin 0.06))
-    (pad 2 smd rect (at -0.7 0) (size 0.35 0.25) (layers F.Cu F.Paste F.Mask)
-      (net 2 GND) (solder_mask_margin 0.06))
-    (pad 7 smd rect (at 0 0) (size 0.5 1.25) (layers F.Cu F.Paste F.Mask)
-      (net 2 GND))
-    (model ${KIPRJMOD}/hark-kicad/Housings_MLF.pretty/6-pin_1.6x1.6_thin_MLF-6.wrl
-      (at (xyz 0 0 0))
-      (scale (xyz 1 1 1))
-      (rotate (xyz 0 0 90))
-    )
-  )
   (module Wurth:450301014042 (layer F.Cu)
     (at 48.006 26.67)
@@
       (net 3 +5V))
   )
+  (module Housings_MLF:Thin_MLF_6_1.6mm_0.5mm_pitch (layer F.Cu)
+    (at 46.0375 30.48)
+    (fp_text reference U1 (at 0 1.7) (layer F.SilkS) hide
+      (effects (font (size 1 1) (thickness 0.15)))
+    )
+    (fp_text value MIC5353-3.3YMT (at 0 -2.8) (layer F.Fab) hide
+      (effects (font (size 1 1) (thickness 0.15)))
+    )
+    (fp_line (start 0.8 -0.7) (end 0.8 -0.8) (layer F.SilkS) (width 0.15))
+    (fp_line (start 0.8 -0.2) (end 0.8 -0.3) (layer F.SilkS) (width 0.15))
+    (fp_line (start 0.8 0.3) (end 0.8 0.2) (layer F.SilkS) (width 0.15))
+    (fp_line (start 0.8 0.8) (end 0.8 0.7) (layer F.SilkS) (width 0.15))
+    (fp_line (start -0.8 0.7) (end -0.8 0.8) (layer F.SilkS) (width 0.15))
+    (fp_line (start -0.8 0.2) (end -0.8 0.3) (layer F.SilkS) (width 0.15))
+    (fp_line (start -0.8 -0.8) (end -0.8 -0.7) (layer F.SilkS) (width 0.15))
+    (fp_line (start -0.8 -0.3) (end -0.8 -0.2) (layer F.SilkS) (width 0.15))
+    (fp_line (start -1.01 -1) (end -0.99 -1) (layer F.SilkS) (width 0.15))
+    (fp_line (start 0.8 0.8) (end -0.8 0.8) (layer F.SilkS) (width 0.15))
+    (fp_line (start -0.8 -0.8) (end 0.8 -0.8) (layer F.SilkS) (width 0.15))
+    (fp_line (start 1 -1) (end 1 1) (layer F.CrtYd) (width 0.05))
+    (fp_line (start 1 1) (end -1 1) (layer F.CrtYd) (width 0.05))
+    (fp_line (start -1 1) (end -1 -1) (layer F.CrtYd) (width 0.05))
+    (fp_line (start -1 -1) (end 1 -1) (layer F.CrtYd) (width 0.05))
+    (pad 4 smd rect (at 0.7 0.5) (size 0.35 0.25) (layers F.Cu F.Paste F.Mask)
+      (net 15 +3V3))
+    (pad 5 smd rect (at 0.7 0) (size 0.35 0.25) (layers F.Cu F.Paste F.Mask))
+    (pad 6 smd rect (at 0.7 -0.5) (size 0.35 0.25) (layers F.Cu F.Paste F.Mask)
+      (net 27 "Net-(C9-Pad2)"))
+    (pad 3 smd rect (at -0.7 0.5) (size 0.35 0.25) (layers F.Cu F.Paste F.Mask)
+      (net 3 +5V))
+    (pad 1 smd rect (at -0.7 -0.5) (size 0.35 0.25) (layers F.Cu F.Paste F.Mask)
+      (net 3 +5V))
+    (pad 2 smd rect (at -0.7 0) (size 0.35 0.25) (layers F.Cu F.Paste F.Mask)
+      (net 2 GND))
+    (pad 7 smd rect (at 0 0) (size 0.5 1.25) (layers F.Cu F.Paste F.Mask)
+      (net 2 GND))
+    (model ${KIPRJMOD}/hark-kicad/Housings_MLF.pretty/6-pin_1.6x1.6_thin_MLF-6.wrl
+      (at (xyz 0 0 0))
+      (scale (xyz 1 1 1))
+      (rotate (xyz 0 0 90))
+    )
+  )
   (gr_line (start 43.5 36) (end 65.25 36) (layer Edge.Cuts) (width 0.15))
