File: master-board/onizuka.sch (KiCad schematic (older format))
At the start: 30 parts, among them IC1 FT232RQ, IC2 ADCMP371, P1 USB_OTG, P2 FTDI, Q1 Q_PMOS_GSD, SW1 SPDT, U1 MIC5353-3.3YMT

Commit message: Many faffing, new ESP stuff.
Parts:
- P2: footprint Pin_Headers:Pin_Header_Angled_2x06 -> Socket_Strips:Socket_Strip_Angled_2x06
Connections:
- net CTS: now also P2.9 (P9); no longer P2.3 (P3)
- net DCD: now also P2.8 (P8); no longer P2.6 (P6)
- net DSR: now also P2.10 (P10); no longer P2.4 (P4)
- net DTR: now also P2.12 (P12); no longer P2.2 (P2)
- net GND: now also P2.11 (P11); no longer P2.1 (P1)
- net PWROUT: now also P2.7 (P7); no longer P2.5 (P5)
- net RI: now also P2.6 (P6); no longer P2.8 (P8)
- net RTS: now also P2.1 (P1); no longer P2.11 (P11)
- net RXD: now also P2.3 (P3); no longer P2.9 (P9)
- net TXD: now also P2.5 (P5); no longer P2.7 (P7)
Other:
- moved on the sheet: P2

Commit message: Various shuffling, adding farnell part numbers.
Parts:
- IC1: Farnell (none) -> 1146033
- P2: Farnell (none) -> 1668355
- R1, R2, R3, R4, R7, R8: Farnell (none) -> 2498165
- SW1: Farnell (none) -> 2134452
Connections:
- net DTR: now also P2.4 (P4); no longer P2.12 (P12)
Other:
- note added: "Onizuka Connector"
- note added: "Output Voltage Sense"
- note added: "Status LEDs"
- moved on the sheet: P2

Commit message: Final tweaks, more farnell part numbers, BOM, gerbers
Parts:
- C1, C4, C5, C6: Farnell (none) -> 2524677
- C2: Farnell (none) -> 2524674
- C3: Farnell (none) -> 2426952
- C7, C8, C9: Farnell (none) -> 2496813
- D1, D5: Farnell (none) -> 2290329
- D2, D3: Farnell (none) -> 8554609
- D4: Farnell (none) -> 2290330
- P1: Farnell (none) -> 2506104
- R1, R2, R3, R7, R8: Farnell 2498165 -> 1358043
- R4: value 1K -> 1k; Farnell 2498165 -> 1358043
- R5: Farnell (none) -> 1358088
- R6: Farnell (none) -> 1358113
- R9: Farnell (none) -> 1358069
Changed lines of the file:
@@
 F 2 "Connect:USB_Micro-B" V 850 950 50  0001 C CNN
 F 3 "" V 850 950 50  0000 C CNN
+F 4 "2506104" H 900 1050 60  0001 C CNN "Farnell"
 	1    900  1050
 	0    -1   1    0
@@
 F 2 "Capacitors_SMD:C_0402" H 2700 2650 50  0001 C CNN
 F 3 "" H 2700 2650 50  0000 C CNN
+F 4 "2524677" H 2700 2650 60  0001 C CNN "Farnell"
 	1    2700 2650
 	1    0    0    -1
@@
 F 2 "LEDs:LED_0603" V 5250 1000 50  0001 C CNN
 F 3 "" V 5250 1000 50  0000 C CNN
+F 4 "2290329" H 5250 1000 60  0001 C CNN "Farnell"
 	1    5250 1000
 	0    -1   -1   0
@@
 F 2 "Resistors_SMD:R_0402" H 5250 1200 50  0001 C CNN
 F 3 "" H 5250 1200 50  0000 C CNN
-F 4 "2498165" H 5250 1200 60  0001 C CNN "Farnell"
+F 4 "1358043" H 5250 1200 60  0001 C CNN "Farnell"
 	1    5250 1200
 	1    0    0    -1
@@
 F 2 "LEDs:LED_0603" V 6350 1000 50  0001 C CNN
 F 3 "" V 6350 1000 50  0000 C CNN
+F 4 "8554609" H 6350 1000 60  0001 C CNN "Farnell"
 	1    6350 1000
 	0    -1   -1   0
@@
 F 2 "Resistors_SMD:R_0402" H 6350 1200 50  0001 C CNN
 F 3 "" H 6350 1200 50  0000 C CNN
-F 4 "2498165" H 6350 1200 60  0001 C CNN "Farnell"
+F 4 "1358043" H 6350 1200 60  0001 C CNN "Farnell"
 	1    6350 1200
 	1    0    0    -1
@@
 F 2 "LEDs:LED_0603" V 5850 1000 50  0001 C CNN
 F 3 "" V 5850 1000 50  0000 C CNN
+F 4 "8554609" H 5850 1000 60  0001 C CNN "Farnell"
 	1    5850 1000
 	0    -1   -1   0
@@
 F 2 "Resistors_SMD:R_0402" H 5850 1200 50  0001 C CNN
 F 3 "" H 5850 1200 50  0000 C CNN
-F 4 "2498165" H 5850 1200 60  0001 C CNN "Farnell"
+F 4 "1358043" H 5850 1200 60  0001 C CNN "Farnell"
 	1    5850 1200
 	1    0    0    -1
@@
 F 2 "Capacitors_SMD:C_0402" H 3450 3350 50  0001 C CNN
 F 3 "" H 3450 3350 50  0000 C CNN
+F 4 "2524677" H 3450 3350 60  0001 C CNN "Farnell"
 	1    3450 3350
 	1    0    0    -1
@@
 F 2 "Capacitors_SMD:C_0402" H 3750 3350 50  0001 C CNN
 F 3 "" H 3750 3350 50  0000 C CNN
+F 4 "2524677" H 3750 3350 60  0001 C CNN "Farnell"
 	1    3750 3350
 	1    0    0    -1
@@
 P 3100 3700
 F 0 "R4" H 3130 3720 50  0001 L CNN
-F 1 "1K" H 3150 3700 50  0000 L CNN
+F 1 "1k" H 3150 3700 50  0000 L CNN
 F 2 "Resistors_SMD:R_0402" H 3100 3700 50  0001 C CNN
 F 3 "" H 3100 3700 50  0000 C CNN
-F 4 "2498165" H 3100 3700 60  0001 C CNN "Farnell"
+F 4 "1358043" H 3100 3700 60  0001 C CNN "Farnell"
 	1    3100 3700
 	1    0    0    -1
@@
 F 2 "Capacitors_SMD:C_0402" H 2250 1050 50  0001 C CNN
 F 3 "" H 2250 1050 50  0000 C CNN
+F 4 "2524677" H 2250 1050 60  0001 C CNN "Farnell"
 	1    2250 1050
 	1    0    0    -1
@@
 F 2 "Resistors_SMD:R_0402" H 4950 2950 50  0001 C CNN
 F 3 "" H 4950 2950 50  0000 C CNN
+F 4 "1358088" H 4950 2950 60  0001 C CNN "Farnell"
 	1    4950 2950
 	1    0    0    -1
@@
 F 2 "Resistors_SMD:R_0402" H 4950 3150 50  0001 C CNN
 F 3 "" H 4950 3150 50  0000 C CNN
+F 4 "1358113" H 4950 3150 60  0001 C CNN "Farnell"
 	1    4950 3150
 	1    0    0    -1
@@
 F 2 "Resistors_SMD:R_0402" H 6150 2600 50  0001 C CNN
 F 3 "" H 6150 2600 50  0000 C CNN
-F 4 "2498165" H 6150 2600 60  0001 C CNN "Farnell"
+F 4 "1358043" H 6150 2600 60  0001 C CNN "Farnell"
 	1    6150 2600
 	1    0    0    -1
@@
 F 2 "LEDs:LED_0603" V 6150 2800 50  0001 C CNN
 F 3 "" V 6150 2800 50  0000 C CNN
+F 4 "2290330" H 6150 2800 60  0001 C CNN "Farnell"
 	1    6150 2800
 	0    -1   -1   0
@@
 F 2 "Resistors_SMD:R_0402" H 6200 3000 50  0001 C CNN
 F 3 "" H 6200 3000 50  0000 C CNN
-F 4 "2498165" H 6200 3000 60  0001 C CNN "Farnell"
+F 4 "1358043" H 6200 3000 60  0001 C CNN "Farnell"
 	1    6200 3000
 	1    0    0    -1
@@
 F 2 "LEDs:LED_0603" V 6200 3200 50  0001 C CNN
 F 3 "" V 6200 3200 50  0000 C CNN
+F 4 "2290329" H 6200 3200 60  0001 C CNN "Farnell"
 	1    6200 3200
 	0    -1   -1   0
@@
 F 2 "Resistors_SMD:R_0402" H 2900 3700 50  0001 C CNN
 F 3 "" H 2900 3700 50  0000 C CNN
+F 4 "1358069" H 2900 3700 60  0001 C CNN "Farnell"
 	1    2900 3700
 	1    0    0    -1
@@
 $EndComp
 $Comp
-L GND #PWR019
+L GND #PWR018
 U 1 1 574DAA35
 P 1450 4000
-F 0 "#PWR019" H 1450 3750 50  0001 C CNN
+F 0 "#PWR018" H 1450 3750 50  0001 C CNN
 F 1 "GND" H 1450 3850 50  0000 C CNN
 F 2 "" H 1450 4000 50  0000 C CNN
@@
 	900  3600 900  3400
 $Comp
-L +5V #PWR020
+L +5V #PWR019
 U 1 1 574DAAB9
 P 800 3400
-F 0 "#PWR020" H 800 3250 50  0001 C CNN
+F 0 "#PWR019" H 800 3250 50  0001 C CNN
 F 1 "+5V" H 800 3540 50  0000 C CNN
 F 2 "" H 800 3400 50  0000 C CNN
@@
 F 2 "Capacitors_SMD:C_0402" H 800 3500 50  0001 C CNN
 F 3 "" H 800 3500 50  0000 C CNN
+F 4 "2496813" H 800 3500 60  0001 C CNN "Farnell"
 	1    800  3500
 	1    0    0    -1
@@
 F 2 "Capacitors_SMD:C_0402" H 2000 3700 50  0001 C CNN
 F 3 "" H 2000 3700 50  0000 C CNN
+F 4 "2496813" H 2000 3700 60  0001 C CNN "Farnell"
 	1    2000 3700
 	1    0    0    -1
 $EndComp
 $Comp
-L +3.3V #PWR021
+L +3.3V #PWR020
 U 1 1 574DAE91
 P 2000 3600
-F 0 "#PWR021" H 2000 3450 50  0001 C CNN
+F 0 "#PWR020" H 2000 3450 50  0001 C CNN
 F 1 "+3.3V" H 2000 3740 50  0000 C CNN
 F 2 "" H 2000 3600 50  0000 C CNN
@@
 F 2 "Capacitors_SMD:C_0402" H 2200 3500 50  0001 C CNN
 F 3 "" H 2200 3500 50  0000 C CNN
+F 4 "2496813" H 2200 3500 60  0001 C CNN "Farnell"
 	1    2200 3500
 	-1   0    0    1
@@
 Output Voltage Control
 $Comp
-L +5V #PWR022
+L +5V #PWR021
 U 1 1 574E2783
 P 6150 2500
-F 0 "#PWR022" H 6150 2350 50  0001 C CNN
+F 0 "#PWR021" H 6150 2350 50  0001 C CNN
 F 1 "+5V" H 6150 2640 50  0000 C CNN
 F 2 "" H 6150 2500 50  0000 C CNN
@@
 $EndComp
 $Comp
-L GND #PWR023
+L GND #PWR022
 U 1 1 574E279A
 P 6200 3300
-F 0 "#PWR023" H 6200 3050 50  0001 C CNN
+F 0 "#PWR022" H 6200 3050 50  0001 C CNN
 F 1 "GND" H 6200 3150 50  0000 C CNN
 F 2 "" H 6200 3300 50  0000 C CNN
@@
 $EndComp
 $Comp
-L GND #PWR024
+L GND #PWR023
 U 1 1 574E27B1
 P 4950 3250
-F 0 "#PWR024" H 4950 3000 50  0001 C CNN
+F 0 "#PWR023" H 4950 3000 50  0001 C CNN
 F 1 "GND" H 4950 3100 50  0000 C CNN
 F 2 "" H 4950 3250 50  0000 C CNN
@@
 $EndComp
 $Comp
-L +5V #PWR025
+L +5V #PWR024
 U 1 1 574E27DF
 P 4950 2850
-F 0 "#PWR025" H 4950 2700 50  0001 C CNN
+F 0 "#PWR024" H 4950 2700 50  0001 C CNN
 F 1 "+5V" H 4950 2990 50  0000 C CNN
 F 2 "" H 4950 2850 50  0000 C CNN
@@
 Connection ~ 1650 1300
 $Comp
-L GND #PWR026
+L GND #PWR025
 U 1 1 574E26EE
 P 800 3600
-F 0 "#PWR026" H 800 3350 50  0001 C CNN
+F 0 "#PWR025" H 800 3350 50  0001 C CNN
 F 1 "GND" H 800 3450 50  0000 C CNN
 F 2 "" H 800 3600 50  0000 C CNN
@@
 	800  3400 1000 3400
 $Comp
-L GND #PWR027
+L GND #PWR026
 U 1 1 574E27B3
 P 950 3650
-F 0 "#PWR027" H 950 3400 50  0001 C CNN
+F 0 "#PWR026" H 950 3400 50  0001 C CNN
 F 1 "GND" H 950 3500 50  0000 C CNN
 F 2 "" H 950 3650 50  0000 C CNN
@@
 	2000 3600 1900 3600
 $Comp
-L GND #PWR028
+L GND #PWR027
 U 1 1 574E28D6
 P 2000 3800
-F 0 "#PWR028" H 2000 3550 50  0001 C CNN
+F 0 "#PWR027" H 2000 3550 50  0001 C CNN
 F 1 "GND" H 2000 3650 50  0000 C CNN
 F 2 "" H 2000 3800 50  0000 C CNN
@@
 	2200 3400 1900 3400
 $Comp
-L GND #PWR029
+L GND #PWR028
 U 1 1 574E2962
 P 2200 3600
-F 0 "#PWR029" H 2200 3350 50  0001 C CNN
+F 0 "#PWR028" H 2200 3350 50  0001 C CNN
 F 1 "GND" H 2200 3450 50  0000 C CNN
 F 2 "" H 2200 3600 50  0000 C CNN
@@
 F 2 "Capacitors_SMD:C_0402" H 1650 1050 50  0001 C CNN
 F 3 "" H 1650 1050 50  0000 C CNN
+F 4 "2524674" H 1650 1050 60  0001 C CNN "Farnell"
 	1    1650 1050
 	1    0    0    -1
@@
 F 2 "Capacitors_SMD:C_0402" H 2400 1050 50  0001 C CNN
 F 3 "" H 2400 1050 50  0000 C CNN
+F 4 "2426952" H 2400 1050 60  0001 C CNN "Farnell"
 	1    2400 1050
 	1    0    0    -1
